File: pcb/kyosoc.kicad_pcb (KiCad board)
At the start: 2 copper layers, 286.4 x 94.4 mm, 65 parts, among them SW1 SW_Push, SW10 SW_Push, SW11 SW_Push, SW12 SW_Push, SW13 SW_Push, SW14 SW_Push, SW15 SW_Push, SW16 SW_Push, SW17 SW_Push, SW18 SW_Push, SW19 SW_Push, SW2 SW_Push, SW20 SW_Push, SW21 SW_Push, SW22 SW_Push, SW23 SW_Push, SW24 SW_Push, SW25 SW_Push, SW26 SW_Push, SW27 SW_Push, SW28 SW_Push, SW29 SW_Push, SW3 SW_Push, SW30 SW_Push, SW31 SW_Push, SW32 SW_Push, SW33 SW_Push, SW34 SW_Push, SW35 SW_Push, SW36 SW_Push, SW37 SW_Push, SW38 SW_Push, SW39 SW_Push, SW4 SW_Push, SW40 SW_Push, SW41 SW_Push, SW42 SW_Push, SW43 SW_Push, SW44 SW_Push, SW45 SW_Push, SW46 SW_Push, SW47 SW_Push, SW48 SW_Push, SW49 SW_Push, SW5 SW_Push, SW50 SW_Push, SW51 SW_Push, SW52 SW_Push, SW53 SW_Push, SW54 SW_Push, SW55 SW_Push, SW56 SW_Push, SW57 SW_Push, SW58 SW_Push, SW59 SW_Push, SW6 SW_Push, SW60 SW_Push, SW61 SW_Push, SW7 SW_Push, SW8 SW_Push, SW9 SW_Push, U1 ATmega32U4-AU, Y1 16MHz

Commit message: update pcb size
Other:
- board size 286.4 x 94.4 mm -> 284.4 x 92.4 mm

Commit message: update more shrink pcb
Other:
- board size 284.4 x 92.4 mm -> 282.8 x 90.8 mm
Changed lines of the file:
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@@
       (net 1 "Net-(C1-Pad1)"))
   )
-  (gr_arc (start 7.3 7.3) (end 7.3 6.3) (angle -90) (layer Edge.Cuts) (width 0.05))
-  (gr_arc (start 289.7 7.3) (end 290.7 7.3) (angle -90) (layer Edge.Cuts) (width 0.05))
-  (gr_arc (start 289.7 97.7) (end 289.7 98.7) (angle -90) (layer Edge.Cuts) (width 0.05))
-  (gr_arc (start 7.3 97.7) (end 6.3 97.7) (angle -90) (layer Edge.Cuts) (width 0.05))
-  (gr_line (start 6.3 97.7) (end 6.3 7.3) (layer Edge.Cuts) (width 0.05))
-  (gr_line (start 289.7 98.7) (end 7.3 98.7) (layer Edge.Cuts) (width 0.05))
-  (gr_line (start 290.7 7.3) (end 290.7 97.7) (layer Edge.Cuts) (width 0.05))
-  (gr_line (start 7.3 6.3) (end 289.7 6.3) (layer Edge.Cuts) (width 0.05))
+  (gr_arc (start 8.1 8.1) (end 8.1 7.1) (angle -90) (layer Edge.Cuts) (width 0.05))
+  (gr_arc (start 288.9 8.1) (end 289.9 8.1) (angle -90) (layer Edge.Cuts) (width 0.05))
+  (gr_arc (start 288.9 96.9) (end 288.9 97.9) (angle -90) (layer Edge.Cuts) (width 0.05))
+  (gr_arc (start 8.1 96.9) (end 7.1 96.9) (angle -90) (layer Edge.Cuts) (width 0.05))
+  (gr_line (start 7.1 96.9) (end 7.1 8.1) (layer Edge.Cuts) (width 0.05))
+  (gr_line (start 288.9 97.9) (end 8.1 97.9) (layer Edge.Cuts) (width 0.05))
+  (gr_line (start 289.9 8.1) (end 289.9 96.9) (layer Edge.Cuts) (width 0.05))
+  (gr_line (start 8.1 7.1) (end 288.9 7.1) (layer Edge.Cuts) (width 0.05))
   (segment (start 136.45 62.1) (end 138.9 59.65) (width 0.4) (layer B.Cu) (net 1))
   (segment (start 138.9 59.65) (end 138.9 48.9) (width 0.4) (layer B.Cu) (net 1))

Commit message: update layout
Parts:
- added D1: D_Small, footprint:1N4148W, B.Cu at (21.9, 14.1)
- added D10: D_Small, footprint:1N4148W, B.Cu at (194.7, 14.1)
- added D11: D_Small, footprint:1N4148W, B.Cu at (213.9, 14.1)
- added D12: D_Small, footprint:1N4148W, B.Cu at (233.1, 14.1)
- added D13: D_Small, footprint:1N4148W, B.Cu at (252.3, 14.1)
- added D14: D_Small, footprint:1N4148W, B.Cu at (271.5, 14.1)
- added D15: D_Small, footprint:1N4148W, B.Cu at (290.7, 14.1)
- added D16: D_Small, footprint:1N4148W, B.Cu at (31.5, 33.3)
- added D17: D_Small, footprint:1N4148W, B.Cu at (60.3, 33.3)
- added D18: D_Small, footprint:1N4148W, B.Cu at (79.5, 33.3)
- added D19: D_Small, footprint:1N4148W, B.Cu at (98.7, 33.3)
- added D2: D_Small, footprint:1N4148W, B.Cu at (41.1, 14.1)
- added D20: D_Small, footprint:1N4148W, B.Cu at (117.9, 33.3)
- added D21: D_Small, footprint:1N4148W, B.Cu at (137.1, 33.3)
- added D22: D_Small, footprint:1N4148W, B.Cu at (156.3, 33.3)
- added D23: D_Small, footprint:1N4148W, B.Cu at (175.5, 33.3)
- added D24: D_Small, footprint:1N4148W, B.Cu at (194.7, 33.3)
- added D25: D_Small, footprint:1N4148W, B.Cu at (213.9, 33.3)
- added D26: D_Small, footprint:1N4148W, B.Cu at (233.1, 33.3)
- added D27: D_Small, footprint:1N4148W, B.Cu at (252.3, 33.3)
- added D28: D_Small, footprint:1N4148W, B.Cu at (271.5, 33.3)
- added D29: D_Small, footprint:1N4148W, B.Cu at (290.7, 33.3)
- added D3: D_Small, footprint:1N4148W, B.Cu at (60.3, 14.1)
- added D30: D_Small, footprint:1N4148W, B.Cu at (31.5, 52.5)
- added D31: D_Small, footprint:1N4148W, B.Cu at (60.3, 52.5)
- added D32: D_Small, footprint:1N4148W, B.Cu at (79.5, 52.5)
- added D33: D_Small, footprint:1N4148W, B.Cu at (98.7, 52.5)
- added D34: D_Small, footprint:1N4148W, B.Cu at (117.9, 52.5)
- added D35: D_Small, footprint:1N4148W, B.Cu at (137.1, 52.5)
- added D36: D_Small, footprint:1N4148W, B.Cu at (156.3, 52.5)
- added D37: D_Small, footprint:1N4148W, B.Cu at (175.5, 52.5)
- added D38: D_Small, footprint:1N4148W, B.Cu at (194.7, 52.5)
- added D39: D_Small, footprint:1N4148W, B.Cu at (213.9, 52.5)
- added D4: D_Small, footprint:1N4148W, B.Cu at (79.5, 14.1)
- added D40: D_Small, footprint:1N4148W, B.Cu at (233.1, 52.5)
- added D41: D_Small, footprint:1N4148W, B.Cu at (252.3, 52.5)
- added D42: D_Small, footprint:1N4148W, B.Cu at (281.1, 52.5)
- added D43: D_Small, footprint:1N4148W, B.Cu at (31.5, 71.7)
- added D44: D_Small, footprint:1N4148W, B.Cu at (60.3, 71.7)
- added D45: D_Small, footprint:1N4148W, B.Cu at (79.5, 71.7)
- added D46: D_Small, footprint:1N4148W, B.Cu at (98.7, 71.7)
- added D47: D_Small, footprint:1N4148W, B.Cu at (117.9, 71.7)
- added D48: D_Small, footprint:1N4148W, B.Cu at (137.1, 71.7)
- added D49: D_Small, footprint:1N4148W, B.Cu at (156.3, 71.7)
- added D5: D_Small, footprint:1N4148W, B.Cu at (98.7, 14.1)
- added D50: D_Small, footprint:1N4148W, B.Cu at (175.5, 71.7)
- added D51: D_Small, footprint:1N4148W, B.Cu at (194.7, 71.7)
- added D52: D_Small, footprint:1N4148W, B.Cu at (213.9, 71.7)
- added D53: D_Small, footprint:1N4148W, B.Cu at (233.1, 71.7)
- added D54: D_Small, footprint:1N4148W, B.Cu at (261.9, 71.7)
- added D55: D_Small, footprint:1N4148W, B.Cu at (290.7, 71.7)
- added D56: D_Small, footprint:1N4148W, B.Cu at (79.5, 90.9)
- added D57: D_Small, footprint:1N4148W, B.Cu at (98.7, 90.9)
- added D58: D_Small, footprint:1N4148W, B.Cu at (127.5, 90.9)
- added D59: D_Small, footprint:1N4148W, B.Cu at (165.9, 90.9)
- added D6: D_Small, footprint:1N4148W, B.Cu at (117.9, 14.1)
- added D60: D_Small, footprint:1N4148W, B.Cu at (194.7, 90.9)
- added D61: D_Small, footprint:1N4148W, B.Cu at (213.9, 90.9)
- added D7: D_Small, footprint:1N4148W, B.Cu at (137.1, 14.1)
- added D8: D_Small, footprint:1N4148W, B.Cu at (156.3, 14.1)
- added D9: D_Small, footprint:1N4148W, B.Cu at (175.5, 14.1)
- added J1: USB_C_Receptacle, footprint:TYPE-C-31-M-12, B.Cu at (295.3, 52.5)
- added R1: 5.1k, footprint:Resistor, B.Cu at (198.4, 120.6)
- added R2: 5.1k, footprint:Resistor, B.Cu at (185.4, 114.4)
- added R3: 22, footprint:Resistor, B.Cu at (198.4, 114.4)
- added R4: 22, footprint:Resistor, B.Cu at (198.4, 117.5)
- added R5: 10k, footprint:Resistor, B.Cu at (185.4, 120.8)
- SW1, SW10, SW11, SW12, SW13, SW14, SW15, SW16, SW17, SW18, SW19, SW2, SW20, SW21, SW22, SW23, SW24, SW25, SW26, SW27, SW28, SW29, SW3, SW30, SW31, SW32, SW33, SW34, SW35, SW36, SW37, SW38, SW39, SW4, SW40, SW41, SW42, SW43, SW44, SW45, SW46, SW47, SW48, SW49, SW5, SW50, SW51, SW52, SW53, SW54, SW55, SW56, SW57, SW58, SW59, SW6, SW60, SW61, SW7, SW8, SW9: footprint footprint:Cherry-MX -> footprint:Cherry-MX-Kailh-Socket
- moved U1 138.2 mm to (268.5, 90.9), turned to 270 degrees
- moved C2 83.0 mm to (200.5, 126.8), turned to 270 degrees
- moved Y1 80.6 mm to (185.5, 127.8), turned to 180 degrees
- moved C1 58.1 mm to (103.4, 114.1)
- turned SW30 to 0 degrees
- turned SW31 to 0 degrees
- turned SW32 to 0 degrees
- turned SW33 to 0 degrees
- turned SW34 to 0 degrees
- turned SW35 to 0 degrees
- turned SW36 to 0 degrees
- turned SW37 to 0 degrees
- turned SW38 to 0 degrees
- turned SW39 to 0 degrees
- turned SW40 to 0 degrees
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Connections:
- C1 pad 2: (no net) -> GND
- C2 pad 2: (no net) -> GND
- SW1 pad 1: (no net) -> /COL-0
- SW1 pad 2: (no net) -> Net-(D1-Pad1)
- SW10 pad 1: (no net) -> /COL-9
- SW10 pad 2: (no net) -> Net-(D10-Pad1)
- SW11 pad 1: (no net) -> /COL-10
- SW11 pad 2: (no net) -> Net-(D11-Pad1)
- SW12 pad 1: (no net) -> /COL-11
- SW12 pad 2: (no net) -> Net-(D12-Pad1)
- SW13 pad 1: (no net) -> /COL-12
- SW13 pad 2: (no net) -> Net-(D13-Pad1)
- SW14 pad 1: (no net) -> /COL-13
- SW14 pad 2: (no net) -> Net-(D14-Pad1)
- SW15 pad 1: (no net) -> /COL-14
- SW15 pad 2: (no net) -> Net-(D15-Pad1)
- SW16 pad 1: (no net) -> /COL-0
- SW16 pad 2: (no net) -> Net-(D16-Pad1)
- SW17 pad 1: (no net) -> /COL-2
- SW17 pad 2: (no net) -> Net-(D17-Pad1)
- SW18 pad 1: (no net) -> /COL-3
- SW18 pad 2: (no net) -> Net-(D18-Pad1)
- SW19 pad 1: (no net) -> /COL-4
- SW19 pad 2: (no net) -> Net-(D19-Pad1)
- SW2 pad 1: (no net) -> /COL-1
- SW2 pad 2: (no net) -> Net-(D2-Pad1)
- SW20 pad 1: (no net) -> /COL-5
- SW20 pad 2: (no net) -> Net-(D20-Pad1)
- SW21 pad 1: (no net) -> /COL-6
- SW21 pad 2: (no net) -> Net-(D21-Pad1)
- SW22 pad 1: (no net) -> /COL-7
- SW22 pad 2: (no net) -> Net-(D22-Pad1)
- SW23 pad 1: (no net) -> /COL-8
- SW23 pad 2: (no net) -> Net-(D23-Pad1)
- SW24 pad 1: (no net) -> /COL-9
- SW24 pad 2: (no net) -> Net-(D24-Pad1)
- SW25 pad 1: (no net) -> /COL-10
- SW25 pad 2: (no net) -> Net-(D25-Pad1)
- SW26 pad 1: (no net) -> /COL-11
- SW26 pad 2: (no net) -> Net-(D26-Pad1)
- SW27 pad 1: (no net) -> /COL-12
- SW27 pad 2: (no net) -> Net-(D27-Pad1)
- SW28 pad 1: (no net) -> /COL-13
- SW28 pad 2: (no net) -> Net-(D28-Pad1)
- SW29 pad 1: (no net) -> /COL-14
- SW29 pad 2: (no net) -> Net-(D29-Pad1)
- SW3 pad 1: (no net) -> /COL-2
- SW3 pad 2: (no net) -> Net-(D3-Pad1)
- SW30 pad 1: (no net) -> /COL-0
- SW30 pad 2: (no net) -> Net-(D30-Pad1)
- SW31 pad 1: (no net) -> /COL-2
- SW31 pad 2: (no net) -> Net-(D31-Pad1)
- SW32 pad 1: (no net) -> /COL-3
- SW32 pad 2: (no net) -> Net-(D32-Pad1)
- SW33 pad 1: (no net) -> /COL-4
- SW33 pad 2: (no net) -> Net-(D33-Pad1)
- SW34 pad 1: (no net) -> /COL-5
- SW34 pad 2: (no net) -> Net-(D34-Pad1)
- SW35 pad 1: (no net) -> /COL-6
- SW35 pad 2: (no net) -> Net-(D35-Pad1)
- SW36 pad 1: (no net) -> /COL-7
- SW36 pad 2: (no net) -> Net-(D36-Pad1)
- SW37 pad 1: (no net) -> /COL-8
- SW37 pad 2: (no net) -> Net-(D37-Pad1)
- SW38 pad 1: (no net) -> /COL-9
- SW38 pad 2: (no net) -> Net-(D38-Pad1)
- SW39 pad 1: (no net) -> /COL-10
- SW39 pad 2: (no net) -> Net-(D39-Pad1)
- SW4 pad 1: (no net) -> /COL-3
- SW4 pad 2: (no net) -> Net-(D4-Pad1)
- SW40 pad 1: (no net) -> /COL-11
- SW40 pad 2: (no net) -> Net-(D40-Pad1)
- SW41 pad 1: (no net) -> /COL-12
- SW41 pad 2: (no net) -> Net-(D41-Pad1)
- SW42 pad 1: (no net) -> /COL-14
- SW42 pad 2: (no net) -> Net-(D42-Pad1)
- SW43 pad 1: (no net) -> /COL-0
- SW43 pad 2: (no net) -> Net-(D43-Pad1)
- SW44 pad 1: (no net) -> /COL-2
- SW44 pad 2: (no net) -> Net-(D44-Pad1)
- SW45 pad 1: (no net) -> /COL-3
- SW45 pad 2: (no net) -> Net-(D45-Pad1)
- SW46 pad 1: (no net) -> /COL-4
- SW46 pad 2: (no net) -> Net-(D46-Pad1)
- SW47 pad 1: (no net) -> /COL-5
- SW47 pad 2: (no net) -> Net-(D47-Pad1)
- SW48 pad 1: (no net) -> /COL-6
- SW48 pad 2: (no net) -> Net-(D48-Pad1)
- SW49 pad 1: (no net) -> /COL-7
- SW49 pad 2: (no net) -> Net-(D49-Pad1)
- SW5 pad 1: (no net) -> /COL-4
- SW5 pad 2: (no net) -> Net-(D5-Pad1)
- SW50 pad 1: (no net) -> /COL-8
- SW50 pad 2: (no net) -> Net-(D50-Pad1)
- SW51 pad 1: (no net) -> /COL-9
- SW51 pad 2: (no net) -> Net-(D51-Pad1)
- SW52 pad 1: (no net) -> /COL-10
- SW52 pad 2: (no net) -> Net-(D52-Pad1)
- SW53 pad 1: (no net) -> /COL-11
- SW53 pad 2: (no net) -> Net-(D53-Pad1)
- SW54 pad 1: (no net) -> /COL-13
- SW54 pad 2: (no net) -> Net-(D54-Pad1)
- SW55 pad 1: (no net) -> /COL-14
- SW55 pad 2: (no net) -> Net-(D55-Pad1)
- SW56 pad 1: (no net) -> /COL-3
- SW56 pad 2: (no net) -> Net-(D56-Pad1)
- SW57 pad 1: (no net) -> /COL-4
- SW57 pad 2: (no net) -> Net-(D57-Pad1)
- SW58 pad 1: (no net) -> /COL-5
- SW58 pad 2: (no net) -> Net-(D58-Pad1)
- SW59 pad 1: (no net) -> /COL-8
- SW59 pad 2: (no net) -> Net-(D59-Pad1)
- SW6 pad 1: (no net) -> /COL-5
- SW6 pad 2: (no net) -> Net-(D6-Pad1)
- SW60 pad 1: (no net) -> /COL-9
- SW60 pad 2: (no net) -> Net-(D60-Pad1)
- SW61 pad 1: (no net) -> /COL-10
- SW61 pad 2: (no net) -> Net-(D61-Pad1)
- SW7 pad 1: (no net) -> /COL-6
- SW7 pad 2: (no net) -> Net-(D7-Pad1)
- SW8 pad 1: (no net) -> /COL-7
- SW8 pad 2: (no net) -> Net-(D8-Pad1)
- SW9 pad 1: (no net) -> /COL-8
- SW9 pad 2: (no net) -> Net-(D9-Pad1)
- U1 pad 10: (no net) -> /ROW-2
- U1 pad 11: (no net) -> /ROW-1
- U1 pad 12: (no net) -> /COL-12
- U1 pad 13: (no net) -> /RESET
- U1 pad 18: (no net) -> /COL-9
- U1 pad 19: (no net) -> /COL-8
- U1 pad 20: (no net) -> /COL-7
- U1 pad 21: (no net) -> /COL-6
- U1 pad 22: (no net) -> /COL-4
- U1 pad 25: (no net) -> /COL-5
- U1 pad 26: (no net) -> /COL-3
- U1 pad 27: (no net) -> /COL-2
- U1 pad 28: (no net) -> /ROW-0
- U1 pad 29: (no net) -> /COL-14
- U1 pad 3: (no net) -> /D-
- U1 pad 30: (no net) -> /COL-13
- U1 pad 31: (no net) -> /COL-11
- U1 pad 32: (no net) -> /COL-10
- U1 pad 4: (no net) -> /D+
- U1 pad 40: (no net) -> /COL-0
- U1 pad 41: (no net) -> /COL-1
- U1 pad 8: (no net) -> /ROW-4
- U1 pad 9: (no net) -> /ROW-3
Routing:
- net Net-(C1-Pad1): track 20.1 -> 0.00 mm
- net Net-(C2-Pad1): track 19.8 -> 0.00 mm
Other:
- board size 282.8 x 90.8 mm -> 290.8 x 96 mm

Commit message: wiring done without reset switch
Parts:
- added C3: 1u, footprint:1206-3216, B.Cu at (23.7, 80.1)
- C1, C2: footprint footprint:Kondensator-2.5mm -> footprint:1206-3216
- J1: value USB_C_Receptacle -> TYPE-C-31-M-12
- R1, R2, R3, R4, R5: footprint footprint:Resistor -> footprint:1206-3216
- moved J1 293.6 mm to (1.70, 52.5), turned to 270 degrees
- moved U1 244.8 mm to (23.7, 90.9)
- moved R1 198.0 mm to (9.30, 62.1), turned to 90 degrees
- moved R3 195.5 mm to (7.70, 71.7), turned to 90 degrees
- moved R4 193.1 mm to (10.9, 71.7), turned to 90 degrees
- moved R2 190.1 mm to (9.30, 42.9), turned to 270 degrees
- moved R5 167.7 mm to (23.7, 76.5)
- moved C2 152.7 mm to (52.5, 89.3), turned to 0 degrees
- moved Y1 147.3 mm to (42.9, 90.9), turned to 90 degrees
- moved C1 55.3 mm to (52.5, 92.5), turned to 0 degrees
Connections:
- U1 pad 1: (no net) -> /ROW-0
- U1 pad 10: /ROW-2 -> /ROW-3
- U1 pad 11: /ROW-1 -> /COL-2
- U1 pad 12: /COL-12 -> /COL-6
- U1 pad 18: /COL-9 -> /COL-7
- U1 pad 19: /COL-8 -> /COL-11
- U1 pad 20: /COL-7 -> /COL-12
- U1 pad 21: /COL-6 -> /COL-13
- U1 pad 22: /COL-4 -> /COL-14
- U1 pad 25: /COL-5 -> /COL-3
- U1 pad 26: /COL-3 -> /COL-4
- U1 pad 27: /COL-2 -> /COL-5
- U1 pad 28: /ROW-0 -> /COL-8
- U1 pad 29: /COL-14 -> /COL-9
- U1 pad 30: /COL-13 -> /COL-10
- U1 pad 31: /COL-11 -> (no net)
- U1 pad 32: /COL-10 -> /ROW-4
- U1 pad 6: (no net) -> Net-(C3-Pad1)
- U1 pad 8: /ROW-4 -> /ROW-1
- U1 pad 9: /ROW-3 -> /ROW-2
Routing:
- net /ROW-0: track 0.00 -> 360.4 mm, vias 0 -> 2
- net /ROW-1: track 0.00 -> 330.9 mm, vias 0 -> 2
- net /COL-14: track 0.00 -> 323.6 mm, vias 0 -> 8
- net /ROW-2: track 0.00 -> 301.4 mm, vias 0 -> 2
- net /ROW-3: track 0.00 -> 294.8 mm, vias 0 -> 2
- net /COL-13: track 0.00 -> 290.5 mm, vias 0 -> 8
- net /COL-12: track 0.00 -> 276.6 mm, vias 0 -> 6
- net /COL-10: track 0.00 -> 260.2 mm, vias 0 -> 10
- net /COL-11: track 0.00 -> 257.1 mm, vias 0 -> 8
- net /COL-9: track 0.00 -> 240.7 mm, vias 0 -> 10
- net /COL-8: track 0.00 -> 215.5 mm, vias 0 -> 10
- net /ROW-4: track 0.00 -> 207.3 mm, vias 0 -> 2
- net /COL-7: track 0.00 -> 179.9 mm, vias 0 -> 8
- net /COL-5: track 0.00 -> 176.8 mm, vias 0 -> 10
- net /COL-6: track 0.00 -> 158.7 mm, vias 0 -> 8
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- added copper zone on B.Cu, net GND
- added copper zone on F.Cu, net GND
Other:
- outline, holes or cut-outs redrawn

Commit message: add tact-switch
Parts:
- added R6: 10k, footprint:1206-3216, B.Cu at (14.1, 95.4)
- added SW62: RESET, footprint:Tact-Switch, B.Cu at (138.9, 90.9)
Connections:
- U1 pad 33: GND -> Net-(R6-Pad2)
Routing:
- net /RESET: track 13.5 -> 131.0 mm, vias 0 -> 1
- net Net-(R6-Pad2): track 0.00 -> 5.60 mm
- net GND: track 26.1 -> 29.8 mm
- net /ROW-4: track 207.3 -> 208.2 mm
Changed lines of the file:
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@@
     (thickness 1.6)
     (drawings 34)
-    (tracks 1006)
+    (tracks 1016)
     (zones 0)
-    (modules 133)
-    (nets 94)
+    (modules 135)
+    (nets 95)
   )
   (page A4)
@@
   (net 92 "Net-(J1-PadA6)")
   (net 93 "Net-(C3-Pad1)")
+  (net 94 "Net-(R6-Pad2)")
   (net_class Default "これはデフォルトのネット クラスです。"
     (clearance 0.2)
@@
     (add_net "Net-(J1-PadA7)")
     (add_net "Net-(J1-PadB5)")
+    (add_net "Net-(R6-Pad2)")
     (add_net VCC)
   )
+  (module footprint:Tact-Switch (layer B.Cu)
+    (at 138.9 90.9)
+    (fp_text reference SW62 (at 0 0) (layer B.SilkS)
+      (effects (font (size 0.9 0.9) (thickness 0.1)) (justify mirror))
+    )
+    (fp_text value RESET (at 0 -10) (layer B.Fab) hide
+      (effects (font (size 1 1) (thickness 0.15)) (justify mirror))
+    )
+    (fp_line (start -3.1 0.8) (end -3.1 -0.8) (layer B.SilkS) (width 0.1))
+    (fp_line (start 3.1 0.8) (end 3.1 -0.8) (layer B.SilkS) (width 0.1))
+    (fp_circle (center 0 0) (end 1.75 0) (layer B.SilkS) (width 0.1))
+    (pad 2 thru_hole circle (at -3.25 -2.25) (size 1.6 1.6) (drill 1) (layers *.Cu *.Mask)
+      (net 82 /RESET))
+    (pad 2 thru_hole circle (at 3.25 -2.25) (size 1.6 1.6) (drill 1) (layers *.Cu *.Mask)
+      (net 82 /RESET))
+    (pad 1 thru_hole circle (at 3.25 2.25) (size 1.6 1.6) (drill 1) (layers *.Cu *.Mask)
+      (net 4 GND))
+    (pad 1 thru_hole circle (at -3.25 2.25) (size 1.6 1.6) (drill 1) (layers *.Cu *.Mask)
+      (net 4 GND))
+  )
+  (module footprint:1206-3216 (layer B.Cu)
+    (at 14.1 95.4 270)
+    (fp_text reference R6 (at -0.9 2.1 90) (layer B.SilkS)
+      (effects (font (size 0.9 0.9) (thickness 0.1)) (justify left mirror))
+    )
+    (fp_text value 10k (at 0 -5 90) (layer B.Fab) hide
+      (effects (font (size 1 1) (thickness 0.15)) (justify mirror))
+    )
+    (fp_line (start -0.3 -0.9) (end 0.3 -0.9) (layer B.SilkS) (width 0.1))
+    (fp_line (start -0.3 0.9) (end 0.3 0.9) (layer B.SilkS) (width 0.1))
+    (pad 2 smd roundrect (at 1.5 0 270) (size 1.8 1.8) (layers B.Cu B.Paste B.Mask) (roundrect_rratio 0.1)
+      (net 94 "Net-(R6-Pad2)"))
+    (pad 1 smd roundrect (at -1.5 0 270) (size 1.8 1.8) (layers B.Cu B.Paste B.Mask) (roundrect_rratio 0.1)
+      (net 4 GND))
+  )
   (module footprint:TYPE-C-31-M-12 (layer B.Cu)
     (at 1.7 52.5 270)
@@
       (net 3 VCC))
     (pad 33 smd roundrect (at 6 4 270) (size 1.2 0.4) (layers B.Cu B.Paste B.Mask) (roundrect_rratio 0.5)
-      (net 4 GND))
+      (net 94 "Net-(R6-Pad2)"))
     (pad 32 smd roundrect (at 6 3.2 270) (size 1.2 0.4) (layers B.Cu B.Paste B.Mask) (roundrect_rratio 0.5)
       (net 86 /ROW-4))
@@
   (via (at 148.5 42.9) (size 0.8) (drill 0.4) (layers F.Cu B.Cu) (net 4))
   (via (at 148.5 62.1) (size 0.8) (drill 0.4) (layers F.Cu B.Cu) (net 4))
-  (via (at 119.7 83.1) (size 0.8) (drill 0.4) (layers F.Cu B.Cu) (net 4))
+  (via (at 119.7 85.9) (size 0.8) (drill 0.4) (layers F.Cu B.Cu) (net 4))
   (via (at 129.3 62.1) (size 0.8) (drill 0.4) (layers F.Cu B.Cu) (net 4))
   (via (at 129.3 42.9) (size 0.8) (drill 0.4) (layers F.Cu B.Cu) (net 4))
@@
   (via (at 110.1 42.9) (size 0.8) (drill 0.4) (layers F.Cu B.Cu) (net 4))
   (via (at 110.1 62.1) (size 0.8) (drill 0.4) (layers F.Cu B.Cu) (net 4))
-  (via (at 90.9 83.1) (size 0.8) (drill 0.4) (layers F.Cu B.Cu) (net 4))
-  (via (at 71.7 83.1) (size 0.8) (drill 0.4) (layers F.Cu B.Cu) (net 4))
+  (via (at 90.9 85.9) (size 0.8) (drill 0.4) (layers F.Cu B.Cu) (net 4))
+  (via (at 71.7 85.9) (size 0.8) (drill 0.4) (layers F.Cu B.Cu) (net 4))
   (via (at 90.9 23.7) (size 0.8) (drill 0.4) (layers F.Cu B.Cu) (net 4))
   (via (at 90.9 42.9) (size 0.8) (drill 0.4) (layers F.Cu B.Cu) (net 4))
@@
   (segment (start 98.7 10.85) (end 96.95 9.1) (width 0.3) (layer B.Cu) (net 13))
   (segment (start 98.7 12.5) (end 98.7 10.85) (width 0.3) (layer B.Cu) (net 13))
-  (segment (start 83.65 88.4) (end 83.65 74.9) (width 0.3) (layer B.Cu) (net 14))
   (segment (start 83.65 71.7) (end 83.65 74.9) (width 0.3) (layer F.Cu) (net 14))
   (segment (start 83.65 69.2) (end 83.65 71.7) (width 0.3) (layer B.Cu) (net 14))
@@
   (via (at 25.3 92.5) (size 0.8) (drill 0.4) (layers F.Cu B.Cu) (net 14))
   (segment (start 25.3 96.9) (end 25.3 92.5) (width 0.3) (layer B.Cu) (net 14))
-  (via (at 83.65 82.1) (size 0.8) (drill 0.4) (layers F.Cu B.Cu) (net 14))
-  (segment (start 77.35 82.1) (end 83.65 82.1) (width 0.3) (layer F.Cu) (net 14))
-  (segment (start 62.1 82.1) (end 77.35 82.1) (width 0.3) (layer F.Cu) (net 14))
-  (segment (start 25.3 92.5) (end 27.7 92.5) (width 0.3) (layer F.Cu) (net 14))
-  (segment (start 40.1 92.9) (end 42.9 90.1) (width 0.3) (layer F.Cu) (net 14))
-  (segment (start 42.9 90.1) (end 54.1 90.1) (width 0.3) (layer F.Cu) (net 14))
-  (segment (start 54.1 90.1) (end 62.1 82.1) (width 0.3) (layer F.Cu) (net 14))
-  (segment (start 27.7 92.5) (end 28.1 92.9) (width 0.3) (layer F.Cu) (net 14))
-  (segment (start 28.1 92.9) (end 40.1 92.9) (width 0.3) (layer F.Cu) (net 14))
   (segment (start 117.9 10.85) (end 116.15 9.1) (width 0.3) (layer B.Cu) (net 15))
   (segment (start 117.9 12.5) (end 117.9 10.85) (width 0.3) (layer B.Cu) (net 15))
@@
   (segment (start 9.395 55.75) (end 10.12 55.75) (width 0.3) (layer B.Cu) (net 4))
   (segment (start 9.395 49.25) (end 10.12 49.25) (width 0.3) (layer B.Cu) (net 4))
+  (segment (start 14.3 94.1) (end 14.1 93.9) (width 0.3) (layer B.Cu) (net 4))
+  (segment (start 17.7 94.1) (end 14.3 94.1) (width 0.3) (layer B.Cu) (net 4))
   (segment (start 29.7 86.9) (end 30.9 86.9) (width 0.3) (layer B.Cu) (net 18))
   (via (at 30.9 86.9) (size 0.8) (drill 0.4) (layers F.Cu B.Cu) (net 18))
@@
   (segment (start 45.25 74.15) (end 33.3 86.1) (width 0.3) (layer F.Cu) (net 10))
   (segment (start 45.25 71.7) (end 45.25 74.15) (width 0.3) (layer F.Cu) (net 10))
+  (via (at 83.65 82.9) (size 0.8) (drill 0.4) (layers F.Cu B.Cu) (net 14))
+  (segment (start 83.65 82.9) (end 83.65 74.9) (width 0.3) (layer B.Cu) (net 14))
+  (segment (start 83.65 88.4) (end 83.65 82.9) (width 0.3) (layer B.Cu) (net 14))
+  (segment (start 27.7 92.5) (end 25.3 92.5) (width 0.3) (layer F.Cu) (net 14))
+  (segment (start 61.3 82.9) (end 54.1 90.1) (width 0.3) (layer F.Cu) (net 14))
+  (segment (start 83.65 82.9) (end 61.3 82.9) (width 0.3) (layer F.Cu) (net 14))
+  (segment (start 54.1 90.1) (end 42.9 90.1) (width 0.3) (layer F.Cu) (net 14))
+  (segment (start 42.9 90.1) (end 40.1 92.9) (width 0.3) (layer F.Cu) (net 14))
+  (segment (start 40.1 92.9) (end 28.1 92.9) (width 0.3) (layer F.Cu) (net 14))
+  (segment (start 28.1 92.9) (end 27.7 92.5) (width 0.3) (layer F.Cu) (net 14))
   (segment (start 30.1 17.3) (end 36.5 17.3) (width 0.3) (layer B.Cu) (net 81))
   (segment (start 42.9 15.7) (end 47.7 15.7) (width 0.3) (layer B.Cu) (net 81))
@@
   (segment (start 31.5 71.9) (end 31.5 18.7) (width 0.3) (layer F.Cu) (net 81))
   (segment (start 31.5 18.7) (end 30.1 17.3) (width 0.3) (layer F.Cu) (net 81))
+  (segment (start 135.65 88.65) (end 142.15 88.65) (width 0.3) (layer B.Cu) (net 82))
+  (segment (start 135.65 88.65) (end 129.1 82.1) (width 0.3) (layer F.Cu) (net 82))
+  (segment (start 129.1 82.1) (end 62.1 82.1) (width 0.3) (layer F.Cu) (net 82))
+  (segment (start 29.7 87.7) (end 39.7 87.7) (width 0.3) (layer B.Cu) (net 82))
+  (via (at 62.1 82.1) (size 0.8) (drill 0.4) (layers F.Cu B.Cu) (net 82))
+  (segment (start 39.7 87.7) (end 45.3 82.1) (width 0.3) (layer B.Cu) (net 82))
+  (segment (start 45.3 82.1) (end 62.1 82.1) (width 0.3) (layer B.Cu) (net 82))
   (segment (start 25.3 84.9) (end 25.3 83.7) (width 0.3) (layer B.Cu) (net 83))
   (via (at 25.3 83.7) (size 0.8) (drill 0.4) (layers F.Cu B.Cu) (net 83))
@@
   (segment (start 79.5 92.5) (end 86.1 92.5) (width 0.3) (layer B.Cu) (net 86))
   (segment (start 98.7 92.5) (end 95.7 92.5) (width 0.3) (layer B.Cu) (net 86))
-  (segment (start 162.9 92.5) (end 165.9 92.5) (width 0.3) (layer B.Cu) (net 86))
-  (segment (start 161.3 94.1) (end 162.9 92.5) (width 0.3) (layer B.Cu) (net 86))
-  (segment (start 154.9 94.1) (end 161.3 94.1) (width 0.3) (layer B.Cu) (net 86))
-  (segment (start 127.5 92.5) (end 153.3 92.5) (width 0.3) (layer B.Cu) (net 86))
-  (segment (start 153.3 92.5) (end 154.9 94.1) (width 0.3) (layer B.Cu) (net 86))
   (segment (start 105.3 92.5) (end 98.7 92.5) (width 0.3) (layer B.Cu) (net 86))
   (segment (start 114.9 92.5) (end 105.3 92.5) (width 0.3) (layer B.Cu) (net 86))
@@
   (segment (start 22.5 97.7) (end 79.5 97.7) (width 0.3) (layer F.Cu) (net 86))
   (segment (start 79.5 97.7) (end 79.5 92.5) (width 0.3) (layer B.Cu) (net 86))
+  (segment (start 162.9 92.5) (end 165.9 92.5) (width 0.3) (layer B.Cu) (net 86))
+  (segment (start 160.1 95.3) (end 162.9 92.5) (width 0.3) (layer B.Cu) (net 86))
+  (segment (start 132.1 95.3) (end 160.1 95.3) (width 0.3) (layer B.Cu) (net 86))
+  (segment (start 129.3 92.5) (end 132.1 95.3) (width 0.3) (layer B.Cu) (net 86))
+  (segment (start 127.5 92.5) (end 129.3 92.5) (width 0.3) (layer B.Cu) (net 86))
   (segment (start 12.4 73.2) (end 10.9 73.2) (width 0.3) (layer B.Cu) (net 87))
   (segment (start 22.1 82.9) (end 12.4 73.2) (width 0.3) (layer B.Cu) (net 87))
@@
   (segment (start 23.7 81.6) (end 25.2 80.1) (width 0.3) (layer B.Cu) (net 93))
   (segment (start 23.7 84.9) (end 23.7 81.6) (width 0.3) (layer B.Cu) (net 93))
+  (segment (start 19.7 96.9) (end 14.1 96.9) (width 0.3) (layer B.Cu) (net 94))
   (zone (net 4) (net_name GND) (layer B.Cu) (hatch edge 0.508)
     (connect_pads (clearance 0.3))
